Commit message: Finished updating references to nuturtle pkg

File: nuturtle_description/urdf/turtlebot3_burger.urdf.xacro (robot description, xacro)
@@ -12,5 +12,5 @@
       <origin xyz="-0.032 0 0.0" rpy="0 0 0"/>
       <geometry>
-        <mesh filename="package://turtlebot3_description/meshes/bases/burger_base.stl" scale="0.001 0.001 0.001"/>
+        <mesh filename="package://nuturtle_description/meshes/burger_base.stl" scale="0.001 0.001 0.001"/>
       </geometry>
       <material name="light_black"/>
@@ -40,5 +40,5 @@
       <origin xyz="0 0 0" rpy="1.57 0 0"/>
       <geometry>
-        <mesh filename="package://turtlebot3_description/meshes/wheels/left_tire.stl" scale="0.001 0.001 0.001"/>
+        <mesh filename="package://nuturtle_description/meshes/left_tire.stl" scale="0.001 0.001 0.001"/>
       </geometry>
       <material name="dark"/>
@@ -68,5 +68,5 @@
       <origin xyz="0 0 0" rpy="1.57 0 0"/>
       <geometry>
-        <mesh filename="package://turtlebot3_description/meshes/wheels/right_tire.stl" scale="0.001 0.001 0.001"/>
+        <mesh filename="package://nuturtle_description/meshes/right_tire.stl" scale="0.001 0.001 0.001"/>
       </geometry>
       <material name="dark"/>
@@ -121,5 +121,5 @@
       <origin xyz="0 0 0.0" rpy="0 0 0"/>
       <geometry>
-        <mesh filename="package://turtlebot3_description/meshes/sensors/lds.stl" scale="0.001 0.001 0.001"/>
+        <mesh filename="package://nuturtle_description/meshes/sensors/lds.stl" scale="0.001 0.001 0.001"/>
       </geometry>
       <material name="dark"/>

Commit message: Added reliance on yaml params in urdf

File: nuturtle_description/urdf/turtlebot3_burger.urdf.xacro (robot description, xacro)
@@ -2,4 +2,8 @@
 <robot name="turtlebot3_burger" xmlns:xacro="http://ros.org/wiki/xacro">
   <xacro:include filename="$(find nuturtle_description)/urdf/common_properties.xacro"/>
+  <xacro:property name="diff_yaml" value="$(find nuturtle_description)/config/diff_params.yaml"/>
+  <xacro:property name="props" value="${load_yaml(diff_yaml)}"/>
+  <xacro:property name="wheel_radius" value="${props['wheel_radius']}"/>
+  <xacro:property name="track_width" value="${props['track_width']}"/>
   <link name="base_footprint"/>
   <joint name="base_joint" type="fixed">
@@ -33,5 +37,5 @@
     <parent link="base_link"/>
     <child link="wheel_left_link"/>
-    <origin xyz="0.0 0.08 0.023" rpy="-1.57 0 0"/>
+    <origin xyz="0.0 ${track_width/2} 0.023" rpy="-1.57 0 0"/>
     <axis xyz="0 0 1"/>
   </joint>
@@ -47,5 +51,5 @@
       <origin xyz="0 0 0" rpy="0 0 0"/>
       <geometry>
-        <cylinder length="0.018" radius="0.033"/>
+        <cylinder length="0.018" radius="${wheel_radius}"/>
       </geometry>
     </collision>
@@ -61,5 +65,5 @@
     <parent link="base_link"/>
     <child link="wheel_right_link"/>
-    <origin xyz="0.0 -0.080 0.023" rpy="-1.57 0 0"/>
+    <origin xyz="0.0 -${track_width/2} 0.023" rpy="-1.57 0 0"/>
     <axis xyz="0 0 1"/>
   </joint>
@@ -75,5 +79,5 @@
       <origin xyz="0 0 0" rpy="0 0 0"/>
       <geometry>
-        <cylinder length="0.018" radius="0.033"/>
+        <cylinder length="0.018" radius="${wheel_radius}"/>
       </geometry>
     </collision>

Commit message: Added color condition in urdf

File: nuturtle_description/urdf/turtlebot3_burger.urdf.xacro (robot description, xacro)
@@ -6,140 +6,152 @@
   <xacro:property name="wheel_radius" value="${props['wheel_radius']}"/>
   <xacro:property name="track_width" value="${props['track_width']}"/>
-  <link name="base_footprint"/>
-  <joint name="base_joint" type="fixed">
-    <parent link="base_footprint"/>
-    <child link="base_link"/>
-    <origin xyz="0.0 0.0 0.010" rpy="0 0 0"/>
-  </joint>
-  <link name="base_link">
-    <visual>
-      <origin xyz="-0.032 0 0.0" rpy="0 0 0"/>
-      <geometry>
-        <mesh filename="package://nuturtle_description/meshes/burger_base.stl" scale="0.001 0.001 0.001"/>
-      </geometry>
-      <material name="light_black"/>
-    </visual>
-    <collision>
-      <origin xyz="-0.032 0 0.070" rpy="0 0 0"/>
-      <geometry>
-        <box size="0.140 0.140 0.143"/>
-      </geometry>
-    </collision>
-    <inertial>
-      <origin xyz="0 0 0" rpy="0 0 0"/>
-      <mass value="8.2573504e-01"/>
-      <inertia ixx="2.2124416e-03" ixy="-1.2294101e-05" ixz="3.4938785e-05"
-               iyy="2.1193702e-03" iyz="-5.0120904e-06"
-               izz="2.0064271e-03" />
-    </inertial>
-  </link>
-  <joint name="wheel_left_joint" type="continuous">
-    <parent link="base_link"/>
-    <child link="wheel_left_link"/>
-    <origin xyz="0.0 ${track_width/2} 0.023" rpy="-1.57 0 0"/>
-    <axis xyz="0 0 1"/>
-  </joint>
-  <link name="wheel_left_link">
-    <visual>
-      <origin xyz="0 0 0" rpy="1.57 0 0"/>
-      <geometry>
-        <mesh filename="package://nuturtle_description/meshes/left_tire.stl" scale="0.001 0.001 0.001"/>
-      </geometry>
-      <material name="dark"/>
-    </visual>
-    <collision>
-      <origin xyz="0 0 0" rpy="0 0 0"/>
-      <geometry>
-        <cylinder length="0.018" radius="${wheel_radius}"/>
-      </geometry>
-    </collision>
-    <inertial>
-      <origin xyz="0 0 0" />
-      <mass value="2.8498940e-02" />
-      <inertia ixx="1.1175580e-05" ixy="-4.2369783e-11" ixz="-5.9381719e-09"
-               iyy="1.1192413e-05" iyz="-1.4400107e-11"
-               izz="2.0712558e-05" />
+  <xacro:arg name="color" default="black"/>
+  <xacro:macro name="bot_color" params="color">
+    <link name="${color}_base_footprint"/>
+    <joint name="${color}_base_joint" type="fixed">
+      <parent link="${color}_base_footprint"/>
+      <child link="${color}_base_link"/>
+      <origin xyz="0.0 0.0 0.010" rpy="0 0 0"/>
+    </joint>
+    <link name="${color}_base_link">
+      <visual>
+        <origin xyz="-0.032 0 0.0" rpy="0 0 0"/>
+        <geometry>
+          <mesh filename="package://nuturtle_description/meshes/burger_base.stl" scale="0.001 0.001 0.001"/>
+        </geometry>
+        <material name="light_black"/>
+      </visual>
+      <collision>
+        <origin xyz="-0.032 0 0.070" rpy="0 0 0"/>
+        <geometry>
+          <box size="0.140 0.140 0.143"/>
+        </geometry>
+      </collision>
+      <inertial>
+        <origin xyz="0 0 0" rpy="0 0 0"/>
+        <mass value="8.2573504e-01"/>
+        <inertia ixx="2.2124416e-03" ixy="-1.2294101e-05" ixz="3.4938785e-05"
+                iyy="2.1193702e-03" iyz="-5.0120904e-06"
+                izz="2.0064271e-03" />
       </inertial>
-  </link>
-  <joint name="wheel_right_joint" type="continuous">
-    <parent link="base_link"/>
-    <child link="wheel_right_link"/>
-    <origin xyz="0.0 -${track_width/2} 0.023" rpy="-1.57 0 0"/>
-    <axis xyz="0 0 1"/>
-  </joint>
-  <link name="wheel_right_link">
-    <visual>
-      <origin xyz="0 0 0" rpy="1.57 0 0"/>
-      <geometry>
-        <mesh filename="package://nuturtle_description/meshes/right_tire.stl" scale="0.001 0.001 0.001"/>
-      </geometry>
-      <material name="dark"/>
-    </visual>
-    <collision>
-      <origin xyz="0 0 0" rpy="0 0 0"/>
-      <geometry>
-        <cylinder length="0.018" radius="${wheel_radius}"/>
-      </geometry>
-    </collision>
-    <inertial>
-      <origin xyz="0 0 0" />
-      <mass value="2.8498940e-02" />
-      <inertia ixx="1.1175580e-05" ixy="-4.2369783e-11" ixz="-5.9381719e-09"
-               iyy="1.1192413e-05" iyz="-1.4400107e-11"
-               izz="2.0712558e-05" />
+    </link>
+    <joint name="wheel_left_joint" type="continuous">
+      <parent link="${color}_base_link"/>
+      <child link="${color}_wheel_left_link"/>
+      <origin xyz="0.0 ${track_width/2} 0.023" rpy="-1.57 0 0"/>
+      <axis xyz="0 0 1"/>
+    </joint>
+    <link name="${color}_wheel_left_link">
+      <visual>
+        <origin xyz="0 0 0" rpy="1.57 0 0"/>
+        <geometry>
+          <mesh filename="package://nuturtle_description/meshes/left_tire.stl" scale="0.001 0.001 0.001"/>
+        </geometry>
+        <material name="dark"/>
+      </visual>
+      <collision>
+        <origin xyz="0 0 0" rpy="0 0 0"/>
+        <geometry>
+          <cylinder length="0.018" radius="${wheel_radius}"/>
+        </geometry>
+      </collision>
+      <inertial>
+        <origin xyz="0 0 0" />
+        <mass value="2.8498940e-02" />
+        <inertia ixx="1.1175580e-05" ixy="-4.2369783e-11" ixz="-5.9381719e-09"
+                iyy="1.1192413e-05" iyz="-1.4400107e-11"
+                izz="2.0712558e-05" />
+        </inertial>
+    </link>
+    <joint name="${color}_wheel_right_joint" type="continuous">
+      <parent link="${color}_base_link"/>
+      <child link="${color}_wheel_right_link"/>
+      <origin xyz="0.0 -${track_width/2} 0.023" rpy="-1.57 0 0"/>
+      <axis xyz="0 0 1"/>
+    </joint>
+    <link name="${color}_wheel_right_link">
+      <visual>
+        <origin xyz="0 0 0" rpy="1.57 0 0"/>
+        <geometry>
+          <mesh filename="package://nuturtle_description/meshes/right_tire.stl" scale="0.001 0.001 0.001"/>
+        </geometry>
+        <material name="dark"/>
+      </visual>
+      <collision>
+        <origin xyz="0 0 0" rpy="0 0 0"/>
+        <geometry>
+          <cylinder length="0.018" radius="${wheel_radius}"/>
+        </geometry>
+      </collision>
+      <inertial>
+        <origin xyz="0 0 0" />
+        <mass value="2.8498940e-02" />
+        <inertia ixx="1.1175580e-05" ixy="-4.2369783e-11" ixz="-5.9381719e-09"
+                iyy="1.1192413e-05" iyz="-1.4400107e-11"
+                izz="2.0712558e-05" />
+        </inertial>
+    </link>
+    <joint name="${color}_caster_back_joint" type="fixed">
+      <parent link="${color}_base_link"/>
+      <child link="${color}_caster_back_link"/>
+      <origin xyz="-0.081 0 -0.004" rpy="-1.57 0 0"/>
+    </joint>
+    <link name="${color}_caster_back_link">
+      <collision>
+        <origin xyz="0 0.001 0" rpy="0 0 0"/>
+        <geometry>
+          <box size="0.030 0.009 0.020"/>
+        </geometry>
+      </collision>
+      <inertial>
+        <origin xyz="0 0 0" />
+        <mass value="0.005" />
+        <inertia ixx="0.001" ixy="0.0" ixz="0.0"
+                iyy="0.001" iyz="0.0"
+                izz="0.001" />
       </inertial>
-  </link>
-  <joint name="caster_back_joint" type="fixed">
-    <parent link="base_link"/>
-    <child link="caster_back_link"/>
-    <origin xyz="-0.081 0 -0.004" rpy="-1.57 0 0"/>
-  </joint>
-  <link name="caster_back_link">
-    <collision>
-      <origin xyz="0 0.001 0" rpy="0 0 0"/>
-      <geometry>
-        <box size="0.030 0.009 0.020"/>
-      </geometry>
-    </collision>
-    <inertial>
-      <origin xyz="0 0 0" />
-      <mass value="0.005" />
-      <inertia ixx="0.001" ixy="0.0" ixz="0.0"
-               iyy="0.001" iyz="0.0"
-               izz="0.001" />
-    </inertial>
-  </link>
-  <joint name="imu_joint" type="fixed">
-    <parent link="base_link"/>
-    <child link="imu_link"/>
-    <origin xyz="-0.032 0 0.068" rpy="0 0 0"/>
-  </joint>
-  <link name="imu_link"/>
-  <joint name="scan_joint" type="fixed">
-    <parent link="base_link"/>
-    <child link="base_scan"/>
-    <origin xyz="-0.032 0 0.172" rpy="0 0 0"/>
-  </joint>
-  <link name="base_scan">
-    <visual>
-      <origin xyz="0 0 0.0" rpy="0 0 0"/>
-      <geometry>
-        <mesh filename="package://nuturtle_description/meshes/sensors/lds.stl" scale="0.001 0.001 0.001"/>
-      </geometry>
-      <material name="dark"/>
-    </visual>
-    <collision>
-      <origin xyz="0.015 0 -0.0065" rpy="0 0 0"/>
-      <geometry>
-        <cylinder length="0.0315" radius="0.055"/>
-      </geometry>
-    </collision>
-    <inertial>
-      <mass value="0.114" />
-      <origin xyz="0 0 0" />
-      <inertia ixx="0.001" ixy="0.0" ixz="0.0"
-               iyy="0.001" iyz="0.0"
-               izz="0.001" />
-    </inertial>
-  </link>
+    </link>
+    <joint name="${color}_imu_joint" type="fixed">
+      <parent link="${color}_base_link"/>
+      <child link="${color}_imu_link"/>
+      <origin xyz="-0.032 0 0.068" rpy="0 0 0"/>
+    </joint>
+    <link name="${color}_imu_link"/>
+    <joint name="${color}_scan_joint" type="fixed">
+      <parent link="${color}_base_link"/>
+      <child link="${color}_base_scan"/>
+      <origin xyz="-0.032 0 0.172" rpy="0 0 0"/>
+    </joint>
+    <link name="${color}_base_scan">
+      <visual>
+        <origin xyz="0 0 0.0" rpy="0 0 0"/>
+        <geometry>
+          <mesh filename="package://nuturtle_description/meshes/sensors/lds.stl" scale="0.001 0.001 0.001"/>
+        </geometry>
+        <material name="dark"/>
+      </visual>
+      <collision>
+        <origin xyz="0.015 0 -0.0065" rpy="0 0 0"/>
+        <geometry>
+          <cylinder length="0.0315" radius="0.055"/>
+        </geometry>
+      </collision>
+      <inertial>
+        <mass value="0.114" />
+        <origin xyz="0 0 0" />
+        <inertia ixx="0.001" ixy="0.0" ixz="0.0"
+                iyy="0.001" iyz="0.0"
+                izz="0.001" />
+      </inertial>
+    </link>
+  </xacro:macro>
+  <xacro:unless value="$(arg color)=='all'">
+    <xacro:bot_color color="$(arg color)"/>
+  </xacro:unless>
+  <xacro:if value="$(arg color)=='all'">
+    <xacro:bot_color color="black"/>
+    <xacro:bot_color color="red"/>
+    <xacro:bot_color color="blue"/>
+    <xacro:bot_color color="green"/>
+  </xacro:if>
 </robot>

Commit message: Changed color of base link

File: nuturtle_description/urdf/turtlebot3_burger.urdf.xacro (robot description, xacro)
@@ -20,5 +20,5 @@
           <mesh filename="package://nuturtle_description/meshes/burger_base.stl" scale="0.001 0.001 0.001"/>
         </geometry>
-        <material name="light_black"/>
+        <material name="$(arg color)"/>
       </visual>
       <collision>

Commit message: Added color as xacro property

File: nuturtle_description/urdf/turtlebot3_burger.urdf.xacro (robot description, xacro)
@@ -7,4 +7,5 @@
   <xacro:property name="track_width" value="${props['track_width']}"/>
   <xacro:arg name="color" default="black"/>
+  <xacro:property name="color" value="$(arg color)"/>
   <xacro:macro name="bot_color" params="color">
     <link name="${color}_base_footprint"/>
@@ -127,5 +128,5 @@
         <origin xyz="0 0 0.0" rpy="0 0 0"/>
         <geometry>
-          <mesh filename="package://nuturtle_description/meshes/sensors/lds.stl" scale="0.001 0.001 0.001"/>
+          <mesh filename="package://nuturtle_description/meshes/lds.stl" scale="0.001 0.001 0.001"/>
         </geometry>
         <material name="dark"/>
@@ -146,8 +147,8 @@
     </link>
   </xacro:macro>
-  <xacro:unless value="$(arg color)=='all'">
-    <xacro:bot_color color="$(arg color)"/>
+  <xacro:unless value="${color == 'all'}">
+    <xacro:bot_color color="${color}"/>
   </xacro:unless>
-  <xacro:if value="$(arg color)=='all'">
+  <xacro:if value="${color == 'all'}">
     <xacro:bot_color color="black"/>
     <xacro:bot_color color="red"/>

Commit message: Removed deprecated xacro prefix

File: nuturtle_description/urdf/turtlebot3_burger.urdf.xacro (robot description, xacro)
@@ -3,5 +3,5 @@
   <xacro:include filename="$(find nuturtle_description)/urdf/common_properties.xacro"/>
   <xacro:property name="diff_yaml" value="$(find nuturtle_description)/config/diff_params.yaml"/>
-  <xacro:property name="props" value="${load_yaml(diff_yaml)}"/>
+  <xacro:property name="props" value="${xacro.load_yaml(diff_yaml)}"/>
   <xacro:property name="wheel_radius" value="${props['wheel_radius']}"/>
   <xacro:property name="track_width" value="${props['track_width']}"/>

Commit message: Modified to take collision radius param

File: nuturtle_description/urdf/turtlebot3_burger.urdf.xacro (robot description, xacro)
@@ -6,4 +6,5 @@
   <xacro:property name="wheel_radius" value="${props['wheel_radius']}"/>
   <xacro:property name="track_width" value="${props['track_width']}"/>
+  <xacro:property name="collision_radius" value="${props['collision_radius']}"/>
   <xacro:arg name="color" default="black"/>
   <xacro:property name="color" value="$(arg color)"/>
@@ -23,10 +24,20 @@
         <material name="$(arg color)"/>
       </visual>
-      <collision>
-        <origin xyz="-0.032 0 0.070" rpy="0 0 0"/>
-        <geometry>
-          <box size="0.140 0.140 0.143"/>
-        </geometry>
-      </collision>
+      <xacro:if value="${collision_radius == 0}">
+        <collision>
+          <origin xyz="-0.032 0 0.070" rpy="0 0 0"/>
+          <geometry>
+            <box size="0.140 0.140 0.143"/>
+          </geometry>
+        </collision>
+      </xacro:if>
+      <xacro:if value="${collision_radius != 0}">
+        <collision>
+          <origin xyz="-0.032 0 0.070" rpy="0 0 0"/>
+          <geometry>
+            <cylinder length=".23" radius="${collision_radius}"/>
+          </geometry>
+        </collision>
+      </xacro:if>
       <inertial>
         <origin xyz="0 0 0" rpy="0 0 0"/>

Commit message: Added color prefix to joint

File: nuturtle_description/urdf/turtlebot3_burger.urdf.xacro (robot description, xacro)
@@ -48,5 +48,5 @@
       </inertial>
     </link>
-    <joint name="wheel_left_joint" type="continuous">
+    <joint name="${color}_wheel_left_joint" type="continuous">
       <parent link="${color}_base_link"/>
       <child link="${color}_wheel_left_link"/>
